Commit message: working ik on robot

File: me380_driver/scripts/me380_robot.urdf (robot description, URDF)
Before this commit: robot me380, 7 links, 6 joints
Links:
- added link ee_link; visual box size=0.03 0.03 0.03
- link base_link: mass 1 -> None; geometry visual box size=0.15, 0.15, 0.05
- link link1: mass 0.5 -> None; geometry visual box size=-0.0622 0.03 0.03; visual box size=0.03 0.03 0.2
- link link2: mass 0.8 -> None; geometry visual box size=0.21575 0.03 0.03
- link link3: mass 0.3 -> None; geometry visual box size=0.08 0.03 0.03
- link link4: mass 0.4 -> None; geometry visual box size=0.03 0.03 0.1
- link link5: mass 0.2 -> None; geometry visual box size=0.0 0.03 0.03
- link link6: mass 0.2 -> None; geometry visual box size=0.03 0.03 0.1
Joints:
- added joint ee_fixed: type fixed, parent link6, child ee_link, origin xyz=0 0 -0.1 rpy=0 0 0
- joint joint1: origin xyz=0.0 0 1.0 rpy=0.0 0 0 -> xyz=0 0 0 rpy=0.0 0 0
- joint joint2: origin xyz=-0.2 0 0.0 rpy=1.5707963267948966 0 0 -> xyz=-0.0622 0 0.2 rpy=-1.5707963267948966 0 0
- joint joint3: origin xyz=1.0 0 0.0 rpy=0.0 0 0 -> xyz=0.21575 0 0 rpy=0.0 0 0
- joint joint4: origin xyz=0.2 0 0 rpy=0 1.5707963267948966 0 -> xyz=0.08 0 0 rpy=0 1.5707963267948966 0
- joint joint5: origin xyz=0 0 0.5 rpy= 0 1.5707963267948966 0 -> xyz=0 0 0.1 rpy= 0 1.5707963267948966 0
- joint joint6: origin xyz=-0.3 0 0 rpy= 0 1.5707963267948966 0 -> xyz=-0.0 0 0 rpy= 0 1.5707963267948966 0

Commit message: cleaned up hardware driver code

File: me380_driver/scripts/me380_robot.urdf (robot description, URDF)
Before this commit: robot me380, 8 links, 7 joints
Links:
- link link1: geometry visual box size=-0.0622 0.03 0.03; visual box size=0.03 0.03 0.2391
- link link2: geometry visual box size=0.2355 0.03 0.03
- link link3: geometry visual box size=0.103 0.03 0.03
- link link4: geometry visual box size=0.03 0.03 0.11
- link link6: geometry visual box size=0.03 0.03 0.112
Joints:
- joint ee_fixed: origin xyz=0 0 -0.1 rpy=0 0 0 -> xyz=0 0 -0.112 rpy=0 0 0
- joint joint1: axis 0 0 1 -> 0 0 -1; limit lower=-3.14159 upper=3.14159 effort=10 velocity=1 -> lower=-2.96706 upper=2.96706 effort=10 velocity=1
- joint joint2: axis 0 0 1 -> 0 0 -1; limit lower=-3.14159 upper=3.14159 effort=10 velocity=1 -> lower=-0.08727 upper=3.92699 effort=10 velocity=1; origin xyz=-0.0622 0 0.2 rpy=-1.5707963267948966 0 0 -> xyz=-0.0622 0 0.2391 rpy=-1.5707963267948966 0 0
- joint joint3: axis 0 0 1 -> 0 0 -1; limit lower=-3.14159 upper=3.14159 effort=10 velocity=1 -> lower=-1.74533 upper=1.74533 effort=10 velocity=1; origin xyz=0.21575 0 0 rpy=0.0 0 0 -> xyz=0.2355 0 0 rpy=0.0 0 0
- joint joint4: limit lower=-3.14159 upper=3.14159 effort=10 velocity=1 -> lower=-2.61799 upper=2.61799 effort=10 velocity=1; origin xyz=0.08 0 0 rpy=0 1.5707963267948966 0 -> xyz=0.103 0 0 rpy=0 1.5707963267948966 0
- joint joint5: limit lower=-3.14159 upper=3.14159 effort=10 velocity=1 -> lower=-1.57080 upper=1.57080 effort=10 velocity=1; origin xyz=0 0 0.1 rpy= 0 1.5707963267948966 0 -> xyz=0 0 0.11 rpy= 0 1.5707963267948966 0
- joint joint6: axis 0 0 1 -> 0 0 -1; limit lower=-3.14159 upper=3.14159 effort=10 velocity=1 -> lower=-2.96706 upper=2.96706 effort=10 velocity=1
