Commit message: updated link length to design lock dims

File: me380_driver/urdf/me380_robot.urdf.xacro (robot description, xacro)
@@ -18,17 +18,16 @@
   <xacro:property name="thick" value="0.03"/>
   <!-- Height and offset of slanted shoulder-->
-  <xacro:property name="link1_height" value="0.2"/>
+  <xacro:property name="link1_height" value="0.2391"/>
   <xacro:property name="link1_side_offset" value="-0.0622"/>
   <!-- Elbow (middle piece) length -->
-  <xacro:property name="link2_len" value="0.21575"/>
-  <!-- 3rd to 4th dof length (4th dof is new added dof) -->
-  <xacro:property name="link3_len" value="0.08"/>
-  <xacro:property name="link3_cz" value="${link3_len/2}"/>  <!-- center at 0, 0, 0.5 -->
+  <xacro:property name="link2_len" value="0.2355"/>
+  <!-- 3rd to 4th dof length (4th dof is new added dof) to face of 4th dof -->
+  <xacro:property name="link3_len" value="0.103"/>
   <!-- end of 4th dof to write differential -->
-  <xacro:property name="link4_len" value="0.1"/>
+  <xacro:property name="link4_len" value="0.110"/>
   <!-- placeholder length -->
   <xacro:property name="link5_len" value="0.0"/>
-  <!-- link6: end-effector flange at tip -->
-  <xacro:property name="gripper_len" value="0.1"/>
+  <!-- link6: diff to midl of gripper dist-->
+  <xacro:property name="gripper_len" value="0.112"/>
   <!-- ============ Base ============ -->
   <link name="base_link">

Commit message: added docker container andjoint limits for urdf

File: me380_driver/urdf/me380_robot.urdf.xacro (robot description, xacro)
@@ -47,6 +47,7 @@
     <child link="link1"/>
     <origin xyz="0 0 0" rpy="${alpha1} 0 0"/>
-    <axis xyz="0 0 1"/>
-    <limit lower="-3.14159" upper="3.14159" effort="10" velocity="1"/>
+    <axis xyz="0 0 -1"/>
+    <!-- +-170 deg limits -->
+    <limit lower="-2.96706" upper="2.96706" effort="10" velocity="1"/>
   </joint>
   <link name="link1">
@@ -77,6 +78,6 @@
     <child link="link2"/>
     <origin xyz="${link1_side_offset} 0 ${link1_height}" rpy="${alpha2} 0 0"/>
-    <axis xyz="0 0 1"/>
-    <limit lower="-3.14159" upper="3.14159" effort="10" velocity="1"/>
+    <axis xyz="0 0 -1"/>
+    <limit lower="-0.08727" upper="3.92699" effort="10" velocity="1"/>
   </joint>
   <link name="link2">
@@ -96,6 +97,6 @@
     <child link="link3"/>
     <origin xyz="${link2_len} 0 0" rpy="${alpha3} 0 0"/>
-    <axis xyz="0 0 1"/>
-    <limit lower="-3.14159" upper="3.14159" effort="10" velocity="1"/>
+    <axis xyz="0 0 -1"/>
+    <limit lower="-1.74533" upper="1.74533" effort="10" velocity="1"/>
   </joint>
   <link name="link3">
@@ -116,5 +117,5 @@
     <origin xyz="${link3_len} 0 0" rpy="0 ${alpha4} 0"/>
     <axis xyz="0 0 1"/>
-    <limit lower="-3.14159" upper="3.14159" effort="10" velocity="1"/>
+    <limit lower="-2.61799" upper="2.61799" effort="10" velocity="1"/>
   </joint>
   <link name="link4">
@@ -135,5 +136,5 @@
     <origin xyz="0 0 ${link4_len}" rpy=" 0 ${alpha5} 0"/>
     <axis xyz="0 0 1"/>
-    <limit lower="-3.14159" upper="3.14159" effort="10" velocity="1"/>
+    <limit lower="-1.57080" upper="1.57080" effort="10" velocity="1"/>
   </joint>
   <link name="link5">
@@ -153,6 +154,6 @@
     <child link="link6"/>
     <origin xyz="-${link5_len} 0 0" rpy=" 0 ${alpha6} 0"/>
-    <axis xyz="0 0 1"/>
-    <limit lower="-3.14159" upper="3.14159" effort="10" velocity="1"/>
+    <axis xyz="0 0 -1"/>
+    <limit lower="-2.96706" upper="2.96706" effort="10" velocity="1"/>
   </joint>
   <link name="link6">

Commit message: fixed minor bugs

File: me380_driver/urdf/me380_robot.urdf.xacro (robot description, xacro)
@@ -172,5 +172,5 @@
     <parent link="link6"/>
     <child link="ee_link"/>
-    <origin xyz="0, 0, ${-gripper_len}" rpy="0 0 0"/>
+    <origin xyz="0 0 ${-gripper_len}" rpy="0 0 0"/>
   </joint>
   <link name="ee_link">
