Commit message: updated urdf

File: me380_driver/urdf/me380_robot.urdf (robot description, URDF)
Before this commit: robot me380, 8 links, 7 joints
Links:
- link ee_link: geometry visual box size=0.03 0.03 0.03
- link link1: geometry visual box size=-0.0622 0.03 0.03; visual box size=0.03 0.03 0.2
- link link2: geometry visual box size=0.21575 0.03 0.03
- link link3: geometry visual box size=0.08 0.03 0.03
- link link4: geometry visual box size=0.03 0.03 0.1
- link link5: geometry visual box size=0.0 0.03 0.03
- link link6: geometry visual box size=0.03 0.03 0.1
Joints:
- joint ee_fixed: origin xyz=0, 0, ${-gripper_len} rpy=0 0 0 -> xyz=0 0 -0.1 rpy=0 0 0
- joint joint1: origin xyz=0 0 0 rpy=${alpha1} 0 0 -> xyz=0 0 0 rpy=0.0 0 0
- joint joint2: origin xyz=${link1_side_offset} 0 ${link1_height} rpy=${alpha2} 0 0 -> xyz=-0.0622 0 0.2 rpy=-1.5707963267948966 0 0
- joint joint3: origin xyz=${link2_len} 0 0 rpy=${alpha3} 0 0 -> xyz=0.21575 0 0 rpy=0.0 0 0
- joint joint4: origin xyz=${link3_len} 0 0 rpy=0 ${alpha4} 0 -> xyz=0.08 0 0 rpy=0 1.5707963267948966 0
- joint joint5: origin xyz=0 0 ${link4_len} rpy= 0 ${alpha5} 0 -> xyz=0 0 0.1 rpy= 0 1.5707963267948966 0
- joint joint6: origin xyz=-${link5_len} 0 0 rpy= 0 ${alpha6} 0 -> xyz=-0.0 0 0 rpy= 0 1.5707963267948966 0

Commit message: increase arduino speed limit, updated gripper length

File: me380_driver/urdf/me380_robot.urdf (robot description, URDF)
Before this commit: robot me380, 8 links, 7 joints
Links:
- link link6: geometry visual box size=0.03 0.03 0.207

File: me380_driver/urdf/me380_robot.urdf.xacro (robot description, xacro)
@@ -29,5 +29,5 @@
   <xacro:property name="link5_len" value="0.0"/>
   <!-- link6: diff to midl of gripper dist-->
-  <xacro:property name="gripper_len" value="0.112"/>
+  <xacro:property name="gripper_len" value="0.207"/>
   <!-- ============ Base ============ -->
   <link name="base_link">

Commit message: updated base position

File: me380_driver/urdf/me380_robot.urdf (robot description, URDF)
Before this commit: robot me380, 8 links, 7 joints
Links:
- link link1: geometry visual box size=-0.0622 0.03 0.03; visual box size=0.03 0.03 0.245

File: me380_driver/urdf/me380_robot.urdf.xacro (robot description, xacro)
@@ -18,5 +18,5 @@
   <xacro:property name="thick" value="0.03"/>
   <!-- Height and offset of slanted shoulder-->
-  <xacro:property name="link1_height" value="0.2391"/>
+  <xacro:property name="link1_height" value="0.245"/>
   <xacro:property name="link1_side_offset" value="-0.0622"/>
   <!-- Elbow (middle piece) length -->
